Commit message: Update names

File: description/skratch.urdf.xacro (robot description, xacro)
@@ -22,14 +22,14 @@
         <child link="skratch_base"/>
     </joint>
-    <xacro:kelo_drive_top_part name="front_left_drive_top_part" parent="skratch_base" drive_name="skratch_1_drive" movable_joints="$(arg movable_joints)">
+    <xacro:kelo_drive_top_part name="front_left_drive_top_part" parent="skratch_base" movable_joints="$(arg movable_joints)">
         <origin xyz="0.202 0.118 -0.054" rpy="0.0 0 0.0"/>
     </xacro:kelo_drive_top_part>
-    <xacro:kelo_drive_top_part name="front_right_drive_top_part" parent="skratch_base" drive_name="skratch_2_drive" movable_joints="$(arg movable_joints)">
+    <xacro:kelo_drive_top_part name="front_right_drive_top_part" parent="skratch_base" movable_joints="$(arg movable_joints)">
         <origin xyz="0.202 -0.118 -0.054" rpy="0.0 0 0.0"/>
     </xacro:kelo_drive_top_part>
-    <xacro:kelo_drive_top_part name="rear_left_drive_top_part" parent="skratch_base" drive_name="skratch_3_drive" movable_joints="$(arg movable_joints)">
+    <xacro:kelo_drive_top_part name="rear_left_drive_top_part" parent="skratch_base" movable_joints="$(arg movable_joints)">
         <origin xyz="-0.202  0.118 -0.054" rpy="0.0 0 0.0"/>
     </xacro:kelo_drive_top_part>
-    <xacro:kelo_drive_top_part name="rear_right_drive_top_part" parent="skratch_base" drive_name="skratch_4_drive" movable_joints="$(arg movable_joints)">
+    <xacro:kelo_drive_top_part name="rear_right_drive_top_part" parent="skratch_base" movable_joints="$(arg movable_joints)">
         <origin xyz="-0.202 -0.118 -0.054" rpy="0.0 0 0.0"/>
     </xacro:kelo_drive_top_part>

File: description/skratch_ros.xacro (robot description, xacro)
@@ -36,16 +36,16 @@
             <plugin>gz_ros2_control/GazeboSimSystem</plugin>
         </hardware>
-        <xacro:joint_interface joint_name="skratch_1_drive_pivot_joint"/>
-        <xacro:joint_interface joint_name="skratch_1_drive_left_hub_wheel_joint"/>
-        <xacro:joint_interface joint_name="skratch_1_drive_right_hub_wheel_joint"/>
-        <xacro:joint_interface joint_name="skratch_2_drive_pivot_joint"/>
-        <xacro:joint_interface joint_name="skratch_2_drive_left_hub_wheel_joint"/>
-        <xacro:joint_interface joint_name="skratch_2_drive_right_hub_wheel_joint"/>
-        <xacro:joint_interface joint_name="skratch_3_drive_pivot_joint"/>
-        <xacro:joint_interface joint_name="skratch_3_drive_left_hub_wheel_joint"/>
-        <xacro:joint_interface joint_name="skratch_3_drive_right_hub_wheel_joint"/>
-        <xacro:joint_interface joint_name="skratch_4_drive_pivot_joint"/>
-        <xacro:joint_interface joint_name="skratch_4_drive_left_hub_wheel_joint"/>
-        <xacro:joint_interface joint_name="skratch_4_drive_right_hub_wheel_joint"/>
+        <xacro:joint_interface joint_name="front_left_drive_pivot_joint"/>
+        <xacro:joint_interface joint_name="front_left_drive_left_hub_wheel_joint"/>
+        <xacro:joint_interface joint_name="front_left_drive_right_hub_wheel_joint"/>
+        <xacro:joint_interface joint_name="front_right_drive_pivot_joint"/>
+        <xacro:joint_interface joint_name="front_right_drive_left_hub_wheel_joint"/>
+        <xacro:joint_interface joint_name="front_right_drive_right_hub_wheel_joint"/>
+        <xacro:joint_interface joint_name="rear_left_drive_pivot_joint"/>
+        <xacro:joint_interface joint_name="rear_left_drive_left_hub_wheel_joint"/>
+        <xacro:joint_interface joint_name="rear_left_drive_right_hub_wheel_joint"/>
+        <xacro:joint_interface joint_name="rear_right_drive_pivot_joint"/>
+        <xacro:joint_interface joint_name="rear_right_drive_left_hub_wheel_joint"/>
+        <xacro:joint_interface joint_name="rear_right_drive_right_hub_wheel_joint"/>
         <xacro:arm_joint_interface joint_name="shoulder_joint" initial_position="0"/>
         <xacro:arm_joint_interface joint_name="half_arm_one_joint" initial_position="-1.5"/>

File: description/wheels/kelo_drive_mid.xacro (robot description, xacro)
@@ -32,5 +32,5 @@
 -->
 <robot xmlns:xacro="http://www.ros.org/wiki/xacro">
-    <xacro:macro name="kelo_drive" params="name parent *origin movable_joints:=true">
+    <xacro:macro name="kelo_drive_mid" params="name parent *origin movable_joints:=true">
         <xacro:include filename="$(find skratch_description)/description/wheels/kelo_drive_wheel.xacro"/>
         <link name="${name}_pivot_link">

File: description/wheels/kelo_drive_top_part.xacro (robot description, xacro)
@@ -8,6 +8,6 @@
 -->
 <robot xmlns:xacro="http://www.ros.org/wiki/xacro">
-    <xacro:macro name="kelo_drive_top_part" params="name parent drive_name:=default_drive_name *origin movable_joints:=true">
-        <xacro:include filename="$(find skratch_description)/description/wheels/kelo_drive.xacro" />
+    <xacro:macro name="kelo_drive_top_part" params="name parent *origin movable_joints:=true">
+        <xacro:include filename="$(find skratch_description)/description/wheels/kelo_drive_mid.xacro" />
         <link name="${name}_drive_top_part">
             <visual>
@@ -37,7 +37,7 @@
             <child link="${name}_drive_top_part"/>
         </joint>
-        <xacro:kelo_drive name="${drive_name}" parent="${name}_drive_top_part" movable_joints="${movable_joints}">
+        <xacro:kelo_drive_mid name="${drive_name}" parent="${name}_drive_top_part" movable_joints="${movable_joints}">
             <origin xyz="0 0 -0.09" rpy="0 0 0.0"/>
-        </xacro:kelo_drive>
+        </xacro:kelo_drive_mid>
     </xacro:macro>
 </robot>
